Commit message: initial commit

File: my_robot/urdf/my_robot.xacro (robot description, xacro)
@@ -50,5 +50,5 @@
       <origin xyz="0 0 0" rpy=" 0 0 0"/>
       <geometry>
-        <box size=".45 .2 .2"/>
+        <box size=".45 .2 .1"/>
       </geometry>
     </collision>
@@ -56,5 +56,5 @@
       <origin xyz="0 0 0" rpy=" 0 0 0"/>
       <geometry>
-        <box size=".45 .2 .2"/>
+        <box size=".45 .2 .1"/>
       </geometry>
     </visual>
@@ -62,5 +62,5 @@
       <origin xyz="-0.15 0 -0.05" rpy=" 0 0 0"/>
       <geometry>
-        <sphere radius="0.0599"/>
+        <sphere radius="0.0499"/>
       </geometry>
     </collision>
@@ -68,5 +68,5 @@
       <origin xyz="-0.15 0 -0.05" rpy=" 0 0 0"/>
       <geometry>
-        <sphere radius="0.06"/>
+        <sphere radius="0.05"/>
       </geometry>
     </visual>
@@ -74,5 +74,5 @@
       <origin xyz="0.15 0 -0.05" rpy=" 0 0 0"/>
       <geometry>
-        <sphere radius="0.0599"/>
+        <sphere radius="0.0499"/>
       </geometry>
     </collision>
@@ -80,5 +80,5 @@
       <origin xyz="0.15 0 -0.05" rpy=" 0 0 0"/>
       <geometry>
-        <sphere radius="0.06"/>
+        <sphere radius="0.05"/>
       </geometry>
     </visual>
@@ -100,5 +100,5 @@
       <origin xyz="0 0 0" rpy=" 0 1.5707 1.5707"/>
       <geometry>
-        <cylinder radius=".11" length="0.05"/>
+        <cylinder radius=".1" length="0.05"/>
       </geometry>
     </collision>
@@ -106,5 +106,5 @@
       <origin xyz="0 0 0" rpy=" 0 1.5707 1.5707"/>
       <geometry>
-        <cylinder radius=".11" length="0.05"/>
+        <cylinder radius=".1" length="0.05"/>
       </geometry>
     </visual>
@@ -126,5 +126,5 @@
       <origin xyz="0 0 0" rpy=" 0 1.5707 1.5707"/>
       <geometry>
-        <cylinder radius=".11" length="0.05"/>
+        <cylinder radius=".1" length="0.05"/>
       </geometry>
     </collision>
@@ -132,5 +132,5 @@
       <origin xyz="0 0 0" rpy=" 0 1.5707 1.5707"/>
       <geometry>
-        <cylinder radius=".11" length="0.05"/>
+        <cylinder radius=".1" length="0.05"/>
       </geometry>
     </visual>

Commit message: initial commit

File: my_robot/urdf/my_robot.xacro (robot description, xacro)
@@ -31,5 +31,5 @@
   </joint>
   <joint type="fixed" name="hokuyo_joint">
-    <origin xyz="0.15 0 .1" rpy="0 0 0"/>
+    <origin xyz="0.15 0 .5" rpy="0 0 0"/>
     <child link="hokuyo"/>
     <parent link="chassis"/>

Commit message: initial commit

File: my_robot/urdf/my_robot.xacro (robot description, xacro)
@@ -31,5 +31,5 @@
   </joint>
   <joint type="fixed" name="hokuyo_joint">
-    <origin xyz="0.15 0 .5" rpy="0 0 0"/>
+    <origin xyz="0.15 0 .1" rpy="0 0 0"/>
     <child link="hokuyo"/>
     <parent link="chassis"/>

Commit message: initial commit

File: my_robot/urdf/my_robot.xacro (robot description, xacro)
@@ -1,4 +1,4 @@
 <?xml version='1.0'?>
-<robot name="my_new_robot" xmlns:xacro="http://www.ros.org/wiki/xacro">
+<robot name="my_robot" xmlns:xacro="http://www.ros.org/wiki/xacro">
   <xacro:include filename="$(find my_robot)/urdf/my_robot.gazebo" />
   <link name="robot_footprint"></link>
@@ -50,5 +50,5 @@
       <origin xyz="0 0 0" rpy=" 0 0 0"/>
       <geometry>
-        <box size=".45 .2 .1"/>
+        <box size=".4 .2 .1"/>
       </geometry>
     </collision>
@@ -56,5 +56,5 @@
       <origin xyz="0 0 0" rpy=" 0 0 0"/>
       <geometry>
-        <box size=".45 .2 .1"/>
+        <box size=".4 .2 .1"/>
       </geometry>
     </visual>
